File: Hardware/AquaHub/Mechanical.sch (KiCad schematic (older format))
At the start: 10 parts

Commit message: Many refinements
Connections:
- net labels removed: LIVE, LIVE_IN, NEUTRAL
- wire segments 3 -> 0
Changed lines of the file:
@@
 	1    0    0    -1
 $EndComp
-$Comp
-L power:PWR_FLAG #FLG0101
-U 1 1 5BB7D235
-P 1925 2300
-F 0 "#FLG0101" H 1925 2375 50  0001 C CNN
-F 1 "PWR_FLAG" V 1925 2428 50  0000 L CNN
-F 2 "" H 1925 2300 50  0001 C CNN
-F 3 "~" H 1925 2300 50  0001 C CNN
-	1    1925 2300
-	0    -1   -1   0
-$EndComp
-Wire Wire Line
-	2200 2300 1925 2300
-Text GLabel 1975 2500 2    50   Output ~ 0
-NEUTRAL
-$Comp
-L power:PWR_FLAG #FLG0102
-U 1 1 5BB7D23D
-P 1925 2500
-F 0 "#FLG0102" H 1925 2575 50  0001 C CNN
-F 1 "PWR_FLAG" V 1925 2628 50  0000 L CNN
-F 2 "" H 1925 2500 50  0001 C CNN
-F 3 "~" H 1925 2500 50  0001 C CNN
-	1    1925 2500
-	0    -1   -1   0
-$EndComp
-Wire Wire Line
-	1925 2500 1975 2500
-Text GLabel 1975 2400 2    50   Output ~ 0
-LIVE
-$Comp
-L power:PWR_FLAG #FLG0103
-U 1 1 5BB7D245
-P 1925 2400
-F 0 "#FLG0103" H 1925 2475 50  0001 C CNN
-F 1 "PWR_FLAG" V 1925 2528 50  0000 L CNN
-F 2 "" H 1925 2400 50  0001 C CNN
-F 3 "~" H 1925 2400 50  0001 C CNN
-	1    1925 2400
-	0    -1   -1   0
-$EndComp
-Wire Wire Line
-	1975 2400 1925 2400
-Text Label 2200 2300 2    39   ~ 0
-LIVE_IN
 $EndSCHEMATC

Commit message: Various changes
Other:
- note added: "Panel perforations"
- note removed: "Panel perfs"
Changed lines of the file:
@@
 Panel mounting
 Text Notes 3675 850  0    39   ~ 0
-Panel perfs
+Panel perforations
 $Comp
 L Mechanical:MountingHole MH?
