File: Hardware/AquaHub/AquaHub.kicad_pcb (KiCad board)
At the start: 2 copper layers, 198.1 x 118.7 mm, 43 parts, among them J1 Screw_Terminal, J10 PinHeader4, J11 PinHeader3, J12 PinHeader3, J2 Screw_Terminal, J3 Screw_Terminal, J4 Screw_Terminal, J5 Screw_Terminal, J6 Screw_Terminal, J7 Screw_Terminal, J8 Screw_Terminal, J9 PinHeader3, K1 MT2-C93402, K2 MT2-C93402, K3 MT2-C93402, K4 MT2-C93402, K5 MT2-C93402, K6 MT2-C93402, U1 ESP32-WROVER-I, U2 ACS723, U3 3.3V Reg, U4 TPL7407LA, U5 5V Reg

Commit message: Lots of new stuff
Parts:
- added MH10: MountingHole, AquaFootprints:Breakaway 1mm, F.Cu at (141.6, 62.2)
- added MH5: MountingHole, MountingHole:MountingHole_2.5mm, F.Cu at (204.5, 49.5)
- added MH6: MountingHole, MountingHole:MountingHole_2.5mm, F.Cu at (41.9, 49.5)
- added MH7: MountingHole, AquaFootprints:Breakaway 1mm, F.Cu at (147.3, 62.2)
- added MH8: MountingHole, AquaFootprints:Breakaway 1mm, F.Cu at (145.4, 62.2)
- added MH9: MountingHole, AquaFootprints:Breakaway 1mm, F.Cu at (143.5, 62.2)
- added SW1: SW_Push, Button_Switch_THT:SW_PUSH_6mm_H13mm, F.Cu at (120.0, 50.8)
- added SW2: SW_Push, Button_Switch_THT:SW_PUSH_6mm_H13mm, F.Cu at (107.5, 50.8)
- added SW3: SW_Push, Button_Switch_THT:SW_PUSH_6mm_H13mm, F.Cu at (94.8, 50.8)
- added SW4: SW_Push, Button_Switch_THT:SW_PUSH_6mm_H13mm, F.Cu at (81.9, 50.8)
- added SW5: SW_Push, Button_Switch_THT:SW_PUSH_6mm_H13mm, F.Cu at (69.4, 50.8)
- added SW6: SW_Push, Button_Switch_THT:SW_PUSH_6mm_H13mm, F.Cu at (57.2, 50.8)
- added U6: TCA9534, Package_SO:SOIC-16W_7.5x12.8mm_P1.27mm, B.Cu at (138.4, 50.0)
- D1, D2, D3, D4, D5, D6: footprint LED_THT:LED_D5.0mm-4 -> LED_THT:LED_D5.0mm-4_RGB
- J1, J2, J3, J4, J5, J6, J7, J8: footprint TerminalBlock_WAGO:TerminalBlock_WAGO_236-103_1x03_P5.00mm_45Degree -> AquaFootprints:weidmuller_pm-5.08-3-way
- J11, J12: value PinHeader3 -> Conn_01x06; footprint Connector_PinHeader_2.54mm:PinHeader_1x03_P2.54mm_Vertical -> Connector_IDC:IDC-Header_2x03_P2.54mm_Vertical
- R2, R3: moved to F.Cu
- U1: value ESP32-WROVER-I -> ESP32-WROVER; footprint AquaFootprints:ESP32-WROVER -> Module:Espressif_ESP32_WROVER
- V1: footprint AquaFootprints:RAC01-GB -> Converter_ACDC:Converter_ACDC_RECOM_RAC01-xxSGB_THT
- moved D6 164.5 mm to (52.7, 44.5), turned to 0 degrees
- moved D5 139.1 mm to (65.4, 44.5), turned to 0 degrees
- moved D4 113.7 mm to (78.1, 44.5), turned to 0 degrees
- moved J10 102.3 mm to (194.3, 74.9), turned to 270 degrees
- moved D3 88.3 mm to (90.8, 44.5), turned to 0 degrees
- moved C3 83.6 mm to (198.4, 107.3), turned to 0 degrees
- moved R4 81.5 mm to (198.4, 104.8), turned to 0 degrees
- moved C4 77.3 mm to (188.9, 107.3)
- moved U1 73.4 mm to (189.2, 91.7), turned to 90 degrees
- moved J9 71.4 mm to (147.3, 74.9)
- moved D2 62.9 mm to (103.5, 44.5), turned to 0 degrees
- moved U4 59.8 mm to (165.7, 91.9), turned to 90 degrees
- moved R3 57.0 mm to (149.2, 79.8)
- moved R2 53.9 mm to (142.9, 79.8), turned to 90 degrees
- moved D1 37.6 mm to (116.2, 44.5), turned to 0 degrees
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Connections:
- net POW3 renamed /POW3
- net POW4 renamed /POW4
- net POW5 renamed /POW5
- net POW6 renamed /POW6
- D1 pad 4: PANEL_LEDS -> /Panel_LED
- J1 pad 1: LIVE1 -> NEUTRAL1
- J1 pad 3: NEUTRAL1 -> LIVE1
- J10 pad 2: RX -> TX
- J10 pad 3: TX -> RX
- J11 pad 1: +5V -> GND
- J11 pad 2: PANEL_LEDS -> /Panel_LED
- J11 pad 3: GND -> /Panel_INT
- J12 pad 1: +5V -> GND
- J12 pad 2: PANEL_LEDS -> /Panel_LED
- J12 pad 3: GND -> /Panel_INT
- J2 pad 1: LIVE2 -> NEUTRAL2
- J2 pad 3: NEUTRAL2 -> LIVE2
- J3 pad 1: LIVE3 -> NEUTRAL3
- J3 pad 3: NEUTRAL3 -> LIVE3
- J4 pad 1: LIVE4 -> NEUTRAL4
- J4 pad 3: NEUTRAL4 -> LIVE4
- J5 pad 1: LIVE5 -> NEUTRAL5
- J5 pad 3: NEUTRAL5 -> LIVE5
- J6 pad 1: LIVE6 -> NEUTRAL6
- J6 pad 3: NEUTRAL6 -> LIVE6
- J7 pad 1: NEUTRAL -> LIVE
- J7 pad 3: LIVE -> NEUTRAL
- J8 pad 1: NEUTRAL -> /LIVE_IN
- J8 pad 3: /LIVE_IN -> NEUTRAL
- R2 pad 1: FLOW_SENSE -> /FLOW_SENSE
- R3 pad 2: FLOW_SENSE -> /FLOW_SENSE
- U1 pad 12: PANEL_LEDS -> (no net)
- U1 pad 14: POWER_SENSE -> (no net)
- U1 pad 16: (no net) -> POWER_SENSE
- U1 pad 23: (no net) -> /FLOW_SENSE
- U1 pad 24: (no net) -> /Panel_INT
- U1 pad 26: (no net) -> /Panel_SDA
- U1 pad 29: (no net) -> /Panel_LED
- U1 pad 31: (no net) -> /Panel_SCL
- U1 pad 33: (no net) -> /POW1
- U1 pad 36: (no net) -> /POW2
- U1 pad 37: FLOW_SENSE -> (no net)
- U1 pad 6: POW1 -> (no net)
- U1 pad 7: POW2 -> (no net)
- U4 pad 1: POW1 -> /POW1
- U4 pad 11: RE6 -> RE1
- U4 pad 12: RE5 -> RE2
- U4 pad 13: RE4 -> RE3
- U4 pad 14: RE3 -> RE4
- U4 pad 15: RE2 -> RE5
- U4 pad 16: RE1 -> RE6
- U4 pad 2: POW2 -> /POW2
Routing:
- net /Panel_LED: track 0.00 -> 121.5 mm, vias 0 -> 2
- net /Panel_INT: track 0.00 -> 99.7 mm, vias 0 -> 2
- net /Panel_SCL: track 0.00 -> 95.5 mm, vias 0 -> 2
- net GND: track 384.4 -> 476.5 mm
- net /Panel_SDA: track 0.00 -> 90.3 mm, vias 0 -> 4
- net Net-(SW6-Pad1): track 0.00 -> 89.0 mm
- net Net-(SW5-Pad1): track 0.00 -> 78.1 mm
- net +3V3: track 69.8 -> 146.3 mm, vias 1 -> 3
- net RE3: track 16.2 -> 90.1 mm
- net RE2: track 35.2 -> 106.5 mm
- net Net-(SW4-Pad1): track 0.00 -> 67.3 mm
- net RE1: track 54.3 -> 120.5 mm
- net RE4: track 15.1 -> 81.0 mm
- net PANEL_LEDS: track 62.3 -> 0.00 mm
- net EARTH: track 228.8 -> 169.0 mm
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Other:
- board size 198.1 x 118.7 mm -> 170.2 x 122.6 mm
- net class Default: trace_width 0.25 -> 0.1524; via_dia 0.8 -> 1
- net class MainsRails: via_dia 0.8 -> 1
- rule via_min_size: 0.4 -> 1
- board text added: "ALWAYS_ON"
- board text added: "SUPPLY"
- board text added: "SWITCHED_A"
- board text added: "SWITCHED_B"
- board text added: "SWITCHED_C"
- board text added: "SWITCHED_D"
- board text added: "SWITCHED_E"
- board text added: "SWITCHED_F"
- board text removed: "5V"
- board text removed: "Flow Sensor"
- board text removed: "G"
- board text removed: "Sense"

Commit message: Auto-generated Outputs
Parts:
- removed R4: 10k, Resistor_SMD:R_0805_2012Metric_Pad1.15x1.40mm_HandSolder
- added C5: 10uF, Capacitor_SMD:CP_Elec_6.3x5.4_Nichicon, F.Cu at (88.9, 88.4)
- added C6: 10uF, Capacitor_SMD:CP_Elec_6.3x5.4_Nichicon, F.Cu at (88.9, 99.9)
- added C7: 4.7uF, Capacitor_SMD:CP_Elec_5x5.4, F.Cu at (108.6, 88.6)
- added C8: 4.7uF, Capacitor_SMD:CP_Elec_5x5.4, F.Cu at (108.6, 100.0)
- added J13: Conn_01x02, Connector_PinHeader_1.00mm:PinHeader_1x02_P1.00mm_Vertical, F.Cu at (183.5, 72.7)
- added REF**: OSHW-Logo_11.4x12mm_SilkScreen, Symbol:OSHW-Logo_11.4x12mm_SilkScreen, F.Cu at (74.9, 76.8)
- added REF**: KiCAD Logo, Symbol:Symbol_KiCAD-Logo_CopperAndSilkScreenTop, F.Cu at (74.9, 67.9)
- C1: value 0.1uF -> 100nF
- C2: value 1nF -> 10nF
- J1, J2, J3, J4, J5, J6: value Screw_Terminal -> Screw_Terminal_01x13; footprint AquaFootprints:weidmuller_pm-5.08-3-way -> TerminalBlock_Phoenix:TerminalBlock_Phoenix_PT-1,5-2-5.0-H_1x02_P5.00mm_Horizontal
- J7: value Screw_Terminal -> Screw_Terminal_01x13; footprint AquaFootprints:weidmuller_pm-5.08-3-way -> TerminalBlock_Phoenix:TerminalBlock_Phoenix_PT-1,5-3-5.0-H_1x03_P5.00mm_Horizontal
- J8: footprint AquaFootprints:weidmuller_pm-5.08-3-way -> TerminalBlock_Phoenix:TerminalBlock_Phoenix_PT-1,5-3-5.0-H_1x03_P5.00mm_Horizontal
- R1: value 4.7K -> 6k-100k?
- RV1: footprint Varistor:RV_Disc_D15.5mm_W4.8mm_P7.5mm -> Varistor:RV_Disc_D15.5mm_W6.1mm_P7.5mm
- U1: value ESP32-WROVER -> ESP32-WROOM; footprint Module:Espressif_ESP32_WROVER -> AquaFootprints:ESP32-WROOM
- U2: value ACS723 -> MLX91210KDC-CAS-102-SP
- U3: value 3.3V Reg -> NCP1117DT33G; footprint Package_TO_SOT_SMD:SOT-223-3_TabPin2 -> Package_TO_SOT_SMD:TO-252-3_TabPin2
- U5: value 5V Reg -> NCP1117DT50G; footprint Converter_DCDC:Converter_DCDC_RECOM_R-78E-0.5_THT -> Package_TO_SOT_SMD:TO-252-3_TabPin2
- moved U4 28.0 mm to (140.8, 104.8), turned to 180 degrees
- moved U5 8.95 mm to (98.6, 88.6), turned to 0 degrees
- moved C1 7.27 mm to (164.1, 111.8), turned to 0 degrees
- moved J8 7.24 mm to (178.4, 140.3)
- moved U3 6.37 mm to (98.8, 99.7)
- moved MH4 6.35 mm to (203.2, 148.6)
- moved J7 6.29 mm to (155.6, 140.3)
- moved MH2 5.72 mm to (43.2, 149.2)
- moved U1 5.63 mm to (194.9, 91.8), turned to 270 degrees
- moved J6 5.46 mm to (137.8, 140.3)
- moved J5 5.39 mm to (121.2, 140.3)
- moved J4 5.32 mm to (104.5, 140.3)
- moved J3 5.25 mm to (87.9, 140.3)
- moved J2 5.18 mm to (71.2, 140.3)
- moved J1 5.12 mm to (54.6, 140.3)
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Connections:
- C2 pad 1: POWER_SENSE -> /Power_Sense
- J1 pad 2: EARTH -> LIVE1
- J10 pad 2: TX -> /RX
- J10 pad 3: RX -> /TX
- J2 pad 2: EARTH -> LIVE2
- J3 pad 2: EARTH -> LIVE3
- J4 pad 2: EARTH -> LIVE4
- J5 pad 2: EARTH -> LIVE5
- J6 pad 2: EARTH -> LIVE6
- J7 pad 2: EARTH -> NEUTRAL
- J7 pad 3: NEUTRAL -> EARTH
- R1 pad 1: +5V -> /Power_Sense
- R1 pad 2: Net-(R1-Pad2) -> GND
- U1 pad 10: /POW5 -> /POW4
- U1 pad 11: /POW6 -> /POW3
- U1 pad 12: (no net) -> /POW2
- U1 pad 13: (no net) -> /POW1
- U1 pad 16: POWER_SENSE -> /Power_Sense
- U1 pad 25: (no net) -> Net-(J13-Pad1)
- U1 pad 3: Net-(R4-Pad1) -> (no net)
- U1 pad 33: /POW1 -> (no net)
- U1 pad 34: RX -> /RX
- U1 pad 35: TX -> /TX
- U1 pad 36: /POW2 -> (no net)
- U1 pad 8: /POW3 -> /POW6
- U1 pad 9: /POW4 -> /POW5
- U2 pad 6: Net-(R1-Pad2) -> GND
- U2 pad 7: POWER_SENSE -> /Power_Sense
- U3 pad 1: +12V -> GND
- U3 pad 2: GND -> +3V3
- U3 pad 3: +3V3 -> +12V
- U4 pad 11: RE1 -> RE6
- U4 pad 12: RE2 -> RE5
- U4 pad 13: RE3 -> RE4
- U4 pad 14: RE4 -> RE3
- U4 pad 15: RE5 -> RE2
- U4 pad 16: RE6 -> RE1
- U5 pad 1: +12V -> GND
- U5 pad 2: GND -> +5V
- U5 pad 3: +5V -> +12V
Routing:
- net EARTH: track 169.0 -> 23.6 mm
- net RE5: track 70.8 -> 21.5 mm
- net RE6: track 55.7 -> 7.02 mm
- net RE4: track 81.0 -> 38.8 mm
- net /Power_Sense: track 0.00 -> 41.8 mm, vias 0 -> 3
- net POWER_SENSE: track 36.1 -> 0.00 mm, vias 1 -> 0
- net RE3: track 90.1 -> 56.2 mm
- net RE2: track 106.5 -> 73.0 mm
- net RE1: track 120.5 -> 90.0 mm
- net GND: track 476.5 -> 453.8 mm
- net /POW6: track 29.2 -> 50.8 mm
- net /POW5: track 29.3 -> 50.2 mm
- net /POW4: track 29.3 -> 47.7 mm
- net +3V3: track 146.3 -> 128.9 mm, vias 3 -> 1
- net +12V: track 191.0 -> 174.3 mm, vias 5 -> 3
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Other:
- board size 170.2 x 122.6 mm -> 170.2 x 116.2 mm
- board text added: "AquaHub PowerBoard v1.0"
- board text removed: "ALWAYS_ON"
- board text removed: "SWITCHED_A"
- board text removed: "SWITCHED_B"
- board text removed: "SWITCHED_C"
- board text removed: "SWITCHED_D"
- board text removed: "SWITCHED_E"
- board text removed: "SWITCHED_F"

Commit message: Many refinements
Parts:
- removed J7: Screw_Terminal_01x13, TerminalBlock_Phoenix:TerminalBlock_Phoenix_PT-1,5-3-5.0-H_1x03_P5.00mm_Horizontal
- removed REF**: OSHW-Logo_11.4x12mm_SilkScreen, Symbol:OSHW-Logo_11.4x12mm_SilkScreen
- removed REF**: KiCAD Logo, Symbol:Symbol_KiCAD-Logo_CopperAndSilkScreenTop
- added C9: 1000uF, Capacitor_SMD:CP_Elec_5x4.4, B.Cu at (155.4, 65.6)
- added D7: WS2811, LED_THT:LED_D5.0mm-4_RGB, F.Cu at (153.2, 59.6)
- added D8: Green, LED_SMD:LED_0805_2012Metric_Pad1.15x1.40mm_HandSolder, F.Cu at (145.2, 91.4)
- added D9: Green, LED_SMD:LED_0805_2012Metric_Pad1.15x1.40mm_HandSolder, F.Cu at (145.2, 101.0)
- added D9: Green, LED_SMD:LED_0805_2012Metric_Pad1.15x1.40mm_HandSolder, F.Cu at (145.2, 99.1)
- added D9: Green, LED_SMD:LED_0805_2012Metric_Pad1.15x1.40mm_HandSolder, F.Cu at (145.2, 97.2)
- added D9: Green, LED_SMD:LED_0805_2012Metric_Pad1.15x1.40mm_HandSolder, F.Cu at (145.2, 95.2)
- added D9: Green, LED_SMD:LED_0805_2012Metric_Pad1.15x1.40mm_HandSolder, F.Cu at (145.2, 93.3)
- added F1: 4A, Fuse:Fuseholder_Blade_Mini_Keystone_3568, F.Cu at (170.2, 120.3)
- added J14: PinHeader3, Connector_PinHeader_2.54mm:PinHeader_1x03_P2.54mm_Vertical, F.Cu at (202.8, 132.6)
- added Q1: BSS138, Package_TO_SOT_SMD:SOT-23, F.Cu at (178.1, 107.3)
- added R10: 680R, Resistor_SMD:R_0805_2012Metric_Pad1.15x1.40mm_HandSolder, F.Cu at (150.2, 91.4)
- added R11: 680R, Resistor_SMD:R_0805_2012Metric_Pad1.15x1.40mm_HandSolder, F.Cu at (150.2, 101.0)
- added R11: 680R, Resistor_SMD:R_0805_2012Metric_Pad1.15x1.40mm_HandSolder, F.Cu at (150.2, 99.1)
- added R11: 680R, Resistor_SMD:R_0805_2012Metric_Pad1.15x1.40mm_HandSolder, F.Cu at (150.2, 97.2)
- added R11: 680R, Resistor_SMD:R_0805_2012Metric_Pad1.15x1.40mm_HandSolder, F.Cu at (150.2, 95.2)
- added R11: 680R, Resistor_SMD:R_0805_2012Metric_Pad1.15x1.40mm_HandSolder, F.Cu at (150.2, 93.3)
- added R4: 4.7K, Resistor_SMD:R_0805_2012Metric_Pad1.15x1.40mm_HandSolder, F.Cu at (193.3, 135.1)
- added R5: 10k, Resistor_SMD:R_0805_2012Metric_Pad1.15x1.40mm_HandSolder, F.Cu at (167.9, 82.3)
- added R6: 10k, Resistor_SMD:R_0805_2012Metric_Pad1.15x1.40mm_HandSolder, F.Cu at (195.3, 102.1)
- added R7: 500R, Resistor_SMD:R_0805_2012Metric_Pad1.15x1.40mm_HandSolder, F.Cu at (159.5, 59.8)
- added R8: 10k, Resistor_SMD:R_0805_2012Metric_Pad1.15x1.40mm_HandSolder, F.Cu at (174.5, 107.2)
- added R9: 10k, Resistor_SMD:R_0805_2012Metric_Pad1.15x1.40mm_HandSolder, F.Cu at (172.2, 107.2)
- added TP1: TestPoint, TestPoint:TestPoint_Keystone_5010-5014_Multipurpose, F.Cu at (123.8, 95.9)
- added TP2: TestPoint, TestPoint:TestPoint_Keystone_5010-5014_Multipurpose, F.Cu at (123.8, 91.4)
- added TP3: TestPoint, TestPoint:TestPoint_Keystone_5010-5014_Multipurpose, F.Cu at (123.8, 87.0)
- added TP4: TestPoint, TestPoint:TestPoint_Keystone_5010-5014_Multipurpose, F.Cu at (123.8, 100.3)
- C3, C4, U1, U4, U6: moved to F.Cu
- D1, D2, D3, D4, D5, D6: value NeoPixel -> WS2811
- J1, J2, J3, J4, J5, J6: value Screw_Terminal_01x13 -> Screw_Terminal_01x02
- J10: value PinHeader4 -> PinHeader6; footprint Connector_PinHeader_2.54mm:PinHeader_1x04_P2.54mm_Vertical -> Connector_PinHeader_2.54mm:PinHeader_1x06_P2.54mm_Vertical
- J11, J12: value Conn_01x06 -> IDC_2x3
- J13: value Conn_01x02 -> PinHeader2; footprint Connector_PinHeader_1.00mm:PinHeader_1x02_P1.00mm_Vertical -> Connector_PinHeader_2.54mm:PinHeader_1x02_P2.54mm_Vertical
- J8: value Screw_Terminal -> Screw_Terminal_01x02; footprint TerminalBlock_Phoenix:TerminalBlock_Phoenix_PT-1,5-3-5.0-H_1x03_P5.00mm_Horizontal -> TerminalBlock_Phoenix:TerminalBlock_Phoenix_PT-1,5-2-5.0-H_1x02_P5.00mm_Horizontal
- K1, K2, K3, K4, K5, K6: value MT2-C93402 -> FTR-F1AA012V; footprint AquaFootprints:MT2-C93400 -> AquaFootprints:fujitsu-ftr1-a
- R1: value 6k-100k? -> 10k
- V1: value RAC01-12SGB -> RAC04-12SGB; footprint Converter_ACDC:Converter_ACDC_RECOM_RAC01-xxSGB_THT -> Converter_ACDC:Converter_ACDC_RECOM_RAC04-xxSGB_THT
- moved J9 72.4 mm to (202.8, 121.4), turned to 0 degrees
- moved R2 67.0 mm to (193.3, 124.0), turned to 0 degrees
- moved R3 60.6 mm to (193.3, 121.4), turned to 180 degrees
- moved C3 47.3 mm to (158.4, 82.0), turned to 90 degrees
- moved C4 41.3 mm to (161.7, 81.4), turned to 90 degrees
- moved J12 33.8 mm to (183.5, 61.0)
- moved U6 32.6 mm to (168.1, 63.5), turned to 0 degrees
- moved J13 25.1 mm to (194.7, 95.1), turned to 0 degrees
- moved U4 22.7 mm to (161.7, 95.9)
- moved K5 21.9 mm to (127.3, 133.3), turned to 90 degrees
- moved K4 21.9 mm to (110.5, 133.3), turned to 90 degrees
- moved K6 21.9 mm to (144.0, 133.3), turned to 90 degrees
- moved K2 21.7 mm to (77.5, 133.3), turned to 90 degrees
- moved K3 21.7 mm to (94.0, 133.3), turned to 90 degrees
- moved K1 21.7 mm to (61.0, 133.3), turned to 90 degrees
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Connections:
- net NEUTRAL1 renamed /NEUTRAL1
- net NEUTRAL2 renamed /NEUTRAL2
- net NEUTRAL3 renamed /NEUTRAL3
- net NEUTRAL4 renamed /NEUTRAL4
- net NEUTRAL5 renamed /NEUTRAL5
- net NEUTRAL6 renamed /NEUTRAL6
- C1 pad 1: +5V -> GND
- C1 pad 2: GND -> +5V
- D1 pad 4: /Panel_LED -> Net-(D1-Pad4)
- J1 pad 2: LIVE1 -> /LIVE1
- J10 pad 2: /RX -> /G0
- J10 pad 3: /TX -> /EN
- J10 pad 4: +5V -> /RX
- J13 pad 1: Net-(J13-Pad1) -> /G0
- J2 pad 2: LIVE2 -> /LIVE2
- J3 pad 2: LIVE3 -> /LIVE3
- J4 pad 2: LIVE4 -> /LIVE4
- J5 pad 2: LIVE5 -> /LIVE5
- J6 pad 2: LIVE6 -> /LIVE6
- J8 pad 1: /LIVE_IN -> /NEUTRAL
- J8 pad 2: EARTH -> /UNFUSED_LIVE
- K1 pad 1: RE1 -> /LIVE1
- K1 pad 4: NEUTRAL -> +12V
- K2 pad 1: RE2 -> /LIVE2
- K2 pad 4: NEUTRAL -> +12V
- K3 pad 1: RE3 -> /LIVE3
- K3 pad 4: NEUTRAL -> +12V
- K4 pad 1: RE4 -> /LIVE4
- K4 pad 4: NEUTRAL -> +12V
- K5 pad 1: RE5 -> /LIVE5
- K5 pad 4: NEUTRAL -> +12V
- K6 pad 1: RE6 -> /LIVE6
- K6 pad 4: NEUTRAL -> +12V
- R2 pad 1: /FLOW_SENSE -> /Flow_Sense
- R3 pad 2: /FLOW_SENSE -> /Flow_Sense
- RV1 pad 1: LIVE -> /LIVE
- RV1 pad 2: NEUTRAL -> /NEUTRAL
- U1 pad 10: /POW4 -> /POW2
- U1 pad 12: /POW2 -> /POW4
- U1 pad 13: /POW1 -> /POW5
- U1 pad 14: (no net) -> /POW6
- U1 pad 16: /Power_Sense -> /Panel_LED_33
- U1 pad 23: /FLOW_SENSE -> /Temp_Sense
- U1 pad 24: /Panel_INT -> /Flow_Sense
- U1 pad 25: Net-(J13-Pad1) -> /G0
- U1 pad 26: /Panel_SDA -> (no net)
- U1 pad 29: /Panel_LED -> (no net)
- U1 pad 3: (no net) -> /EN
- U1 pad 31: /Panel_SCL -> (no net)
- U1 pad 37: (no net) -> /Power_Sense
- U1 pad 6: (no net) -> /Panel_INT
- U1 pad 7: (no net) -> /Panel_SDA
- U1 pad 8: /POW6 -> /Panel_SCL
- U1 pad 9: /POW5 -> /POW1
- U2 pad 1: LIVE -> /LIVE
- U2 pad 2: LIVE -> /LIVE
- U4 pad 1: /POW1 -> /POW6
- U4 pad 11: RE6 -> /RE1
- U4 pad 12: RE5 -> /RE2
- U4 pad 13: RE4 -> /RE3
- U4 pad 14: RE3 -> /RE4
- U4 pad 15: RE2 -> /RE5
- U4 pad 16: RE1 -> /RE6
- U4 pad 2: /POW2 -> /POW5
- U4 pad 3: /POW3 -> /POW4
- U4 pad 4: /POW4 -> /POW3
- U4 pad 5: /POW5 -> /POW2
- U4 pad 6: /POW6 -> /POW1
- V1 pad 1: NEUTRAL -> /LIVE
- V1 pad 2: LIVE -> /NEUTRAL
- V1 pad 3: GND -> (no net)
- V1 pad 4: +12V -> GND
Routing:
- net GND: track 453.8 -> 671.0 mm, vias 4 -> 7
- net /NEUTRAL: track 0.00 -> 206.0 mm
- net NEUTRAL: track 205.1 -> 0.00 mm
- net LIVE: track 193.3 -> 0.00 mm
- net /LIVE: track 0.00 -> 185.6 mm
- net /RE1: track 0.00 -> 115.8 mm, vias 0 -> 2
- net /Power_Sense: track 41.8 -> 151.4 mm, vias 3 -> 0
- net +5V: track 316.7 -> 415.5 mm, vias 8 -> 0
- net /RE2: track 0.00 -> 98.2 mm, vias 0 -> 2
- net +12V: track 174.3 -> 266.2 mm, vias 3 -> 0
- net RE1: track 90.0 -> 0.00 mm
- net RE2: track 73.0 -> 0.00 mm
- net /Temp_Sense: track 0.00 -> 70.5 mm
- net /EN: track 0.00 -> 63.7 mm
- net RE3: track 56.2 -> 0.00 mm
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- added copper zone on B.Cu, net GND
- removed copper zone on F.Cu, net GND
Other:
- board size 170.2 x 116.2 mm -> 170 x 100 mm
- board text added: "12V"
- board text added: "3.3V"
- board text added: "4A Fuse"
- board text added: "5V"
- board text added: "A"
- board text added: "B"
- board text added: "C"
- board text added: "Current Sensor"
- board text added: "D"
- board text added: "EN"
- board text added: "F"
- board text added: "FLOW"
- board text added: "G0"
- board text added: "LED Shifter"
- board text added: "Mechanical parts must be on a metric grid."
- board text added: "PROG"
- board text added: "Power Management"
- board text added: "Relay Driver"
- board text added: "STATUS"
- board text added: "SWITCH A"
- board text added: "SWITCH B"
- board text added: "SWITCH C"
- board text added: "SWITCH D"
- board text added: "SWITCH E"
- board text added: "SWITCH F"
- board text added: "TEMP"
- board text added: "UART"
- board text removed: "ISP"

Commit message: Various changes
Parts:
- removed the D9 at (145.2, 101.0)
- removed the D9 at (145.2, 99.1)
- removed the D9 at (145.2, 97.2)
- removed the D9 at (145.2, 95.2)
- removed the D9 at (145.2, 93.3)
- removed R10, R11 (x5): 680R, Resistor_SMD:R_0805_2012Metric_Pad1.15x1.40mm_HandSolder
- added D10: Green, LED_SMD:LED_0603_1608Metric_Pad1.05x0.95mm_HandSolder, F.Cu at (151.6, 96.1)
- added D11: Green, LED_SMD:LED_0603_1608Metric_Pad1.05x0.95mm_HandSolder, F.Cu at (151.6, 98.0)
- added D12: Green, LED_SMD:LED_0603_1608Metric_Pad1.05x0.95mm_HandSolder, F.Cu at (151.6, 99.9)
- added D13: Green, LED_SMD:LED_0603_1608Metric_Pad1.05x0.95mm_HandSolder, F.Cu at (151.6, 101.9)
- added D9: Green, LED_SMD:LED_0603_1608Metric_Pad1.05x0.95mm_HandSolder, F.Cu at (151.6, 94.2)
- added LS1: Piezo, Buzzer_Beeper:Buzzer_12x9.5RM7.6, F.Cu at (193.0, 137.2)
- added RN1: 680R, AquaFootprints:CAT25, F.Cu at (146.2, 97.1)
- C1, C2: footprint Capacitor_SMD:C_0805_2012Metric_Pad1.15x1.40mm_HandSolder -> Capacitor_SMD:C_0603_1608Metric_Pad1.05x0.95mm_HandSolder
- D8: footprint LED_SMD:LED_0805_2012Metric_Pad1.15x1.40mm_HandSolder -> LED_SMD:LED_0603_1608Metric_Pad1.05x0.95mm_HandSolder
- moved J9 12.1 mm to (202.8, 109.3)
- moved R3 12.1 mm to (193.3, 109.3)
- moved J14 12.1 mm to (202.8, 120.5)
- moved R2 12.1 mm to (193.3, 111.9)
- moved R4 12.1 mm to (193.3, 123.1)
- moved D8 6.46 mm to (151.6, 92.3)
- moved C6 1.96 mm to (97.8, 99.9)
- moved J13 0.89 mm to (195.6, 95.1)
- moved U5 0.86 mm to (107.8, 88.6)
- moved U3 0.69 mm to (107.8, 99.7)
- moved C5 0.64 mm to (97.8, 88.4)
Connections:
- net /G0 renamed /IO0
- D8 pad 1: Net-(D8-Pad1) -> /RE1
- D8 pad 2: +12V -> Net-(D8-Pad2)
- U1 pad 23: /Temp_Sense -> (no net)
- U1 pad 24: /Flow_Sense -> (no net)
- U1 pad 26: (no net) -> /Temp_Sense
- U1 pad 27: (no net) -> /Flow_Sense
- U1 pad 28: (no net) -> /Power_Sense
- U1 pad 31: (no net) -> /Panel_INT
- U1 pad 33: (no net) -> /Panel_SDA
- U1 pad 36: (no net) -> /Panel_SCL
- U1 pad 37: /Power_Sense -> /Sounder
- U1 pad 6: /Panel_INT -> (no net)
- U1 pad 7: /Panel_SDA -> (no net)
- U1 pad 8: /Panel_SCL -> (no net)
Routing:
- net /Power_Sense: track 151.4 -> 58.9 mm, vias 0 -> 8
- net /Sounder: track 0.00 -> 72.2 mm
- net /RE5: track 17.9 -> 46.1 mm, vias 0 -> 2
- net /RE4: track 36.0 -> 62.9 mm, vias 0 -> 2
- net /RE3: track 54.2 -> 80.7 mm, vias 0 -> 2
- net /Panel_SCL: track 96.9 -> 118.0 mm
- net /RE6: track 9.34 -> 30.4 mm, vias 0 -> 2
- net /Panel_INT: track 97.8 -> 118.6 mm
- net /Panel_SDA: track 94.0 -> 111.5 mm
- net /Temp_Sense: track 70.5 -> 55.6 mm, vias 0 -> 2
- net +5V: track 415.5 -> 405.5 mm
- net Net-(D8-Pad2): track 0.00 -> 6.85 mm
- net Net-(D13-Pad2): track 0.00 -> 6.82 mm
- net GND: track 671.0 -> 664.6 mm, vias 7 -> 9
- net Net-(D9-Pad2): track 0.00 -> 5.25 mm
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Other:
- board text added: "D8-D12"

Commit message: Various updates and tweaks
Parts:
- C9: value 1000uF -> 220uF; footprint Capacitor_SMD:CP_Elec_5x4.4 -> Capacitor_SMD:CP_Elec_8x6.2
- K1, K2, K3, K4, K5, K6: value FTR-F1AA012V -> 5A Relay; footprint AquaFootprints:fujitsu-ftr1-a -> Relay_THT:Relay_DPST_Fujitsu_FTR-F1A
- R1, R2, R3, R4, R5, R6, R7, R8, R9: footprint Resistor_SMD:R_0805_2012Metric_Pad1.15x1.40mm_HandSolder -> Resistor_SMD:R_0603_1608Metric_Pad1.05x0.95mm_HandSolder
- U1: footprint AquaFootprints:ESP32-WROOM -> Module:Espressif_ESP32_WROOM_32_SMT
- U2: value MLX91210KDC-CAS-102-SP -> Current Sense
- U3: value NCP1117DT33G -> 1A 3.3V
- U4: value TPL7407LA -> Low-Side Driver
- U5: value NCP1117DT50G -> 1A 5V
- U6: footprint Package_SO:SOIC-16W_7.5x12.8mm_P1.27mm -> Package_SO:SOIC-16W_7.5x10.3mm_P1.27mm
- V1: value RAC04-12SGB -> 4W AC-DC Converter; footprint Converter_ACDC:Converter_ACDC_RECOM_RAC04-xxSGB_THT -> Converter_ACDC:Converter_ACDC_RECOM_RAC04-xxSGx_THT
- moved U1 4.27 mm to (180.7, 89.5), turned to 0 degrees
- turned V1 to 90 degrees
Connections:
- K1 pad 4: +12V -> /RE1
- K1 pad 5: /RE1 -> +12V
- K2 pad 4: +12V -> /RE2
- K2 pad 5: /RE2 -> +12V
- K3 pad 4: +12V -> /RE3
- K3 pad 5: /RE3 -> +12V
- K4 pad 4: +12V -> /RE4
- K4 pad 5: /RE4 -> +12V
- K5 pad 4: +12V -> /RE5
- K5 pad 5: /RE5 -> +12V
- K6 pad 4: +12V -> /RE6
- K6 pad 5: /RE6 -> +12V
Routing:
- net GND: track 664.6 -> 676.4 mm
- net /RE4: track 62.9 -> 55.4 mm
- net /RE3: track 80.7 -> 74.0 mm
- net /RE1: track 115.9 -> 109.5 mm
- net /RE2: track 98.2 -> 91.9 mm
- net /RE5: track 46.1 -> 40.4 mm
- net /RE6: track 30.4 -> 25.7 mm
- net +12V: track 263.5 -> 259.8 mm
