File: Hardware/AquaHub/AquaHub.sch (KiCad schematic (older format))
At the start: 37 parts, among them J1 Screw_Terminal, J10 PinHeader4, J11 PinHeader3, J12 PinHeader3, J2 Screw_Terminal, J3 Screw_Terminal, J4 Screw_Terminal, J5 Screw_Terminal, J6 Screw_Terminal, J7 Screw_Terminal, J8 Screw_Terminal, J9 PinHeader3, K1 MT2-C93402, K2 MT2-C93402, K3 MT2-C93402, K4 MT2-C93402, K5 MT2-C93402, K6 MT2-C93402, U1 ESP32-WROVER-I, U2 ACS723, U3 3.3V Reg, U4 TPL7407LA, U5 5V Reg

Commit message: Lots of new stuff
Parts:
- removed J11, J12: PinHeader3, Connector_PinHeader_2.54mm:PinHeader_1x03_P2.54mm_Vertical, symbol Connector_Generic:Conn_01x03
- removed MH1, MH2, MH3, MH4: MountingHole, MountingHole:MountingHole_4.3mm_M4, symbol Mechanical:MountingHole
- removed U1: ESP32-WROVER-I, AquaFootprints:ESP32-WROVER, symbol AquaParts:ESP32-WROVER-I
- added U1: ESP32-WROVER, Module:Espressif_ESP32_WROVER, symbol MCU_Espressif:ESP32-WROVER
- J1, J2, J3, J4, J5, J6, J7, J8: footprint TerminalBlock_WAGO:TerminalBlock_WAGO_236-103_1x03_P5.00mm_45Degree -> AquaFootprints:weidmuller_pm-5.08-3-way
- V1: footprint AquaFootprints:RAC01-GB -> Converter_ACDC:Converter_ACDC_RECOM_RAC01-xxSGB_THT; symbol AquaParts:RAC01-GB -> Converter_ACDC:RAC01-05SGB
Connections:
- net labels added: Panel_INT, Panel_LED, Panel_SCL, Panel_SDA
- net labels removed: PANEL_LEDS
- wire segments 184 -> 180
- no-connect marks 34 -> 31
Other:
- note removed: "13 strapping pin"
- note removed: "23-25\nstrapping pins"
- note removed: "29 strapping pin"

Commit message: Auto-generated Outputs
Parts:
- removed J1, J2, J3, J4, J5, J6: Screw_Terminal, AquaFootprints:weidmuller_pm-5.08-3-way, symbol Connector:Screw_Terminal_01x03
- removed R4: 10k, Resistor_SMD:R_0805_2012Metric_Pad1.15x1.40mm_HandSolder, symbol Device:R_Small
- removed U1: ESP32-WROVER, Module:Espressif_ESP32_WROVER, symbol MCU_Espressif:ESP32-WROVER
- added C5, C6: 10uF, Capacitor_SMD:CP_Elec_6.3x5.4_Nichicon, symbol Device:CP_Small
- added C7, C8: 4.7uF, Capacitor_SMD:CP_Elec_5x5.4, symbol Device:CP_Small
- added J1, J2, J3, J4, J5, J6: Screw_Terminal_01x13, TerminalBlock_Phoenix:TerminalBlock_Phoenix_PT-1,5-2-5.0-H_1x02_P5.00mm_Horizontal, symbol Connector:Screw_Terminal_01x02
- added J13: Conn_01x02, Connector_PinHeader_1.00mm:PinHeader_1x02_P1.00mm_Vertical, symbol Connector_Generic:Conn_01x02
- added U1: ESP32-WROOM, AquaFootprints:ESP32-WROOM, symbol AquaParts:ESP32-WROOM
- C1: value 0.1uF -> 100nF
- C2: value 1nF -> 10nF
- J7: value Screw_Terminal -> Screw_Terminal_01x13; footprint AquaFootprints:weidmuller_pm-5.08-3-way -> TerminalBlock_Phoenix:TerminalBlock_Phoenix_PT-1,5-3-5.0-H_1x03_P5.00mm_Horizontal
- J8: footprint AquaFootprints:weidmuller_pm-5.08-3-way -> TerminalBlock_Phoenix:TerminalBlock_Phoenix_PT-1,5-3-5.0-H_1x03_P5.00mm_Horizontal
- R1: value 4.7K -> 6k-100k?
- RV1: footprint Varistor:RV_Disc_D15.5mm_W4.8mm_P7.5mm -> Varistor:RV_Disc_D15.5mm_W6.1mm_P7.5mm
- U2: value ACS723 -> MLX91210KDC-CAS-102-SP; symbol Sensor_Current:ACS723xLCTR-05AB -> AquaParts:MLX91210
- U3: value 3.3V Reg -> NCP1117DT33G; footprint Package_TO_SOT_SMD:SOT-223-3_TabPin2 -> Package_TO_SOT_SMD:TO-252-3_TabPin2; symbol AquaParts:3.3V-Reg -> Regulator_Linear:NCP1117-3.3_TO252
- U5: value 5V Reg -> NCP1117DT50G; footprint Converter_DCDC:Converter_DCDC_RECOM_R-78E-0.5_THT -> Package_TO_SOT_SMD:TO-252-3_TabPin2; symbol AquaParts:5V-Reg -> Regulator_Linear:NCP1117-5.0_TO252
Connections:
- net labels added: Power_Sense
- net labels removed: POWER_SENSE
- wire segments 180 -> 195
- no-connect marks 31 -> 33
Other:
- note added: "?"
- note added: "Alert Sounder?"
- note added: "Always-On Outputs"
- note added: "Switchable Outputs"
- note added: "Temperature Sensor?"
- note removed: "Main Pump Power"

Commit message: Many refinements
Parts:
- removed J7: Screw_Terminal_01x13, TerminalBlock_Phoenix:TerminalBlock_Phoenix_PT-1,5-3-5.0-H_1x03_P5.00mm_Horizontal, symbol Connector:Screw_Terminal_01x03
- removed J8: Screw_Terminal, TerminalBlock_Phoenix:TerminalBlock_Phoenix_PT-1,5-3-5.0-H_1x03_P5.00mm_Horizontal, symbol Connector:Screw_Terminal_01x03
- added D8, D9, D? (x4): Green, LED_SMD:LED_0805_2012Metric_Pad1.15x1.40mm_HandSolder, symbol Device:LED_Small
- added F1: 4A, Fuse:Fuseholder_Blade_Mini_Keystone_3568, symbol Device:Fuse
- added J14: PinHeader3, Connector_PinHeader_2.54mm:PinHeader_1x03_P2.54mm_Vertical, symbol Connector_Generic:Conn_01x03
- added J8: Screw_Terminal_01x02, TerminalBlock_Phoenix:TerminalBlock_Phoenix_PT-1,5-2-5.0-H_1x02_P5.00mm_Horizontal, symbol Connector:Screw_Terminal_01x02
- added Q1: BSS138, Package_TO_SOT_SMD:SOT-23, symbol Transistor_FET:BSS138
- added R10, R11, R? (x4): 680R, Resistor_SMD:R_0805_2012Metric_Pad1.15x1.40mm_HandSolder, symbol Device:R
- added R4: 4.7K, Resistor_SMD:R_0805_2012Metric_Pad1.15x1.40mm_HandSolder, symbol Device:R
- added R5, R6, R8, R9: 10k, Resistor_SMD:R_0805_2012Metric_Pad1.15x1.40mm_HandSolder, symbol Device:R
- added TP1, TP2, TP3, TP4: TestPoint, TestPoint:TestPoint_Keystone_5010-5014_Multipurpose, symbol Connector:TestPoint
- J1, J2, J3, J4, J5, J6: value Screw_Terminal_01x13 -> Screw_Terminal_01x02
- J10: value PinHeader4 -> PinHeader6; footprint Connector_PinHeader_2.54mm:PinHeader_1x04_P2.54mm_Vertical -> Connector_PinHeader_2.54mm:PinHeader_1x06_P2.54mm_Vertical; symbol Connector_Generic:Conn_01x04 -> Connector_Generic:Conn_01x06
- J13: value Conn_01x02 -> PinHeader2; footprint Connector_PinHeader_1.00mm:PinHeader_1x02_P1.00mm_Vertical -> Connector_PinHeader_2.54mm:PinHeader_1x02_P2.54mm_Vertical
- K1, K2, K3, K4, K5, K6: value MT2-C93402 -> FTR-F1AA012V; footprint AquaFootprints:MT2-C93400 -> AquaFootprints:fujitsu-ftr1-a; symbol AquaParts:MT2-C93402 -> AquaParts:FTR-F1-A
- R1: value 6k-100k? -> 10k
- V1: value RAC01-12SGB -> RAC04-12SGB; footprint Converter_ACDC:Converter_ACDC_RECOM_RAC01-xxSGB_THT -> Converter_ACDC:Converter_ACDC_RECOM_RAC04-xxSGB_THT; symbol Converter_ACDC:RAC01-05SGB -> Converter_ACDC:RAC04-xxGA
Connections:
- net labels added: EN, Flow_Sense, G0, Panel_LED_33, Temp_Sense, UNFUSED_LIVE
- net labels removed: EARTH, FLOW_SENSE
- wire segments 195 -> 277
- no-connect marks 33 -> 19
Other:
- note added: "Logic-Level Shifter"
- note added: "Missing: Alert Sounder\nTo Do: Change pin-headers to terminals\nTo Do: Replace panel board buttons?"
- note added: "Temperature Sensor"
- note added: "These are 240V connectors and\nneed to be rated for at least 2A."
- note added: "This are 240V connector and\nneed to be rated for at least 4A."
- note added: "This connector goes to\nan in-tank DS18B20 \ntemperature sensor"
- note added: "UART"
- note removed: "Air Pump Power"
- note removed: "Alert Sounder?"
- note removed: "Always-On Outputs"
- note removed: "CO2 Power"
- note removed: "Feature Pump Power"
- note removed: "Heater Power"
- note removed: "ISP"
- note removed: "Light A Power"
- note removed: "Light B Power"
- note removed: "Temperature Sensor?"
- moved on the sheet: U3, U5

Commit message: Various changes
Parts:
- removed R10, R11, R? (x4): 680R, Resistor_SMD:R_0805_2012Metric_Pad1.15x1.40mm_HandSolder, symbol Device:R
- added LS1: Piezo, Buzzer_Beeper:Buzzer_12x9.5RM7.6, symbol Device:Speaker_Crystal
- added RN1: 680R, AquaFootprints:CAT25, symbol AquaParts:CAT25
- C1, C2: footprint Capacitor_SMD:C_0805_2012Metric_Pad1.15x1.40mm_HandSolder -> Capacitor_SMD:C_0603_1608Metric_Pad1.05x0.95mm_HandSolder
- D10, D11, D12, D13: renamed from D?; footprint LED_SMD:LED_0805_2012Metric_Pad1.15x1.40mm_HandSolder -> LED_SMD:LED_0603_1608Metric_Pad1.05x0.95mm_HandSolder
- D8, D9: footprint LED_SMD:LED_0805_2012Metric_Pad1.15x1.40mm_HandSolder -> LED_SMD:LED_0603_1608Metric_Pad1.05x0.95mm_HandSolder
Connections:
- net labels added: IO0, Sounder
- net labels removed: G0
- wire segments 277 -> 253
- no-connect marks 19 -> 21
Other:
- note added: "Alert Sounder"
- note added: "All of the 240V load passes\nthrough this component.\nRated at 50A max, reading\nat 40mV/A."
- note added: "Microcontroller"
- note added: "Relay Status Display"
- note added: "The incoming 240V AC mains supply is first\ntaken down to 12V DC, then two regulators\nare used to get a 5V and 3.3V."
- note added: "This is a simple logic level shifter to drive \nthe 5V NeoPixels from the 3.3V signal."
- note added: "Using a relay driver IC means we don't have to\nworry about diodes, and we can drive any size\nrelay from the 3.3V GPIO pins directly."
- moved on the sheet: U3, U5

Commit message: Various updates and tweaks
Parts:
- C1: manf# (none) -> GRM033R61C104ME14D
- C2: manf# (none) -> VJ0603A102GXAPW1BC
- C3: manf# (none) -> TAJB106K006SNJ
- C4: manf# (none) -> TAJD107K006SNJ
- C5, C6: manf# (none) -> UWX1H100MCL1GB
- C7, C8: manf# (none) -> UWX1H4R7MCL1GB
- J1, J2, J3, J4, J5, J6, J8: manf# (none) -> 1935161
- K1, K2, K3, K4, K5, K6: value FTR-F1AA012V -> 5A Relay; footprint AquaFootprints:fujitsu-ftr1-a -> Relay_THT:Relay_DPST_Fujitsu_FTR-F1A; symbol AquaParts:FTR-F1-A -> Relay:Fujitsu_FTR-F1A; manf# (none) -> FTR-F1AA012V
- LS1: manf# (none) -> PS1240P02BT
- Q1: manf# (none) -> BSS138
- R1, R5, R6, R8, R9: footprint Resistor_SMD:R_0805_2012Metric_Pad1.15x1.40mm_HandSolder -> Resistor_SMD:R_0603_1608Metric_Pad1.05x0.95mm_HandSolder; manf# (none) -> GWCR0603-10KFT5
- R2: footprint Resistor_SMD:R_0805_2012Metric_Pad1.15x1.40mm_HandSolder -> Resistor_SMD:R_0603_1608Metric_Pad1.05x0.95mm_HandSolder; manf# (none) -> RC0603JR-072K2L
- R3: footprint Resistor_SMD:R_0805_2012Metric_Pad1.15x1.40mm_HandSolder -> Resistor_SMD:R_0603_1608Metric_Pad1.05x0.95mm_HandSolder; manf# (none) -> GWCR0603-2K2FT5
- R4: footprint Resistor_SMD:R_0805_2012Metric_Pad1.15x1.40mm_HandSolder -> Resistor_SMD:R_0603_1608Metric_Pad1.05x0.95mm_HandSolder; manf# (none) -> GWCR0603-4K7FT5
- RN1: manf# (none) -> CAT25-681JALF
- RV1: manf# (none) -> B72214P2251K101
- U1: footprint AquaFootprints:ESP32-WROOM -> Module:Espressif_ESP32_WROOM_32_SMT; symbol AquaParts:ESP32-WROOM -> MCU_Espressif:ESP32-WROOM-32; manf# (none) -> ESP32-WROOM-32D
- U2: value MLX91210KDC-CAS-102-SP -> Current Sense; manf# (none) -> MLX91210KDC-CAS-102-SP
- U3: value NCP1117DT33G -> 1A 3.3V; manf# (none) -> NCP1117DT33G
- U4: value TPL7407LA -> Low-Side Driver; manf# (none) -> TPL7407LADR
- U5: value NCP1117DT50G -> 1A 5V; manf# (none) -> NCP1117DT50G
- V1: value RAC04-12SGB -> 4W AC-DC Converter; footprint Converter_ACDC:Converter_ACDC_RECOM_RAC04-xxSGB_THT -> Converter_ACDC:Converter_ACDC_RECOM_RAC04-xxSGx_THT; manf# (none) -> RAC04-12SGB
Connections:
- no-connect marks 21 -> 20

Commit message: Before trying a single-board
Parts:
- added Q2: 2SC1815, Package_TO_SOT_SMD:SOT-416, symbol Transistor_BJT:2SC1815
- added R10, R11: 1K, Resistor_SMD:R_0603_1608Metric_Pad1.05x0.95mm_HandSolder, symbol Device:R
- LS1: footprint Buzzer_Beeper:Buzzer_12x9.5RM7.6 -> Buzzer_Beeper:Buzzer_TDK_PS1240P02BT_D12.2mm_H6.5mm
Connections:
- wire segments 253 -> 260
Other:
- moved on the sheet: U3, U5
