File: Hardware/AquaHub/FrontPanel.sch (KiCad schematic (older format))
At the start: 6 parts

Commit message: Lots of new stuff
Parts:
- added J11, J12: Conn_01x06, Connector_IDC:IDC-Header_2x03_P2.54mm_Vertical, symbol Connector_Generic:Conn_01x06
- added SW1, SW2, SW3, SW4, SW5, SW6: SW_Push, Button_Switch_THT:SW_PUSH_6mm_H13mm, symbol Switch:SW_Push
- added U6: TCA9534, Package_SO:SOIC-16W_7.5x12.8mm_P1.27mm, symbol Interface_Expansion:TCA9534
- D1, D2, D3, D4, D5, D6: footprint LED_THT:LED_D5.0mm-4 -> LED_THT:LED_D5.0mm-4_RGB
Connections:
- net labels added: Button_INT, Button_SCL, Button_SDA, Panel_INT, Panel_SCL, Panel_SDA
- net labels removed: 5V
- wire segments 34 -> 95
- no-connect marks 1 -> 3
Other:
- note added: "Indicator LEDs"
- note added: "Input Buttons"
- note added: "Off-board connector"

Commit message: Auto-generated Outputs
Other:
- note added: "?"
Changed lines of the file:
@@
 Text Notes 3650 3600 0    50   ~ 0
 Input Buttons
+Text Notes 5875 4100 0    79   ~ 16
+?
+Text Notes 4025 2150 0    79   ~ 16
+?
+Text Notes 2100 1925 0    79   ~ 16
+?
 $EndSCHEMATC

Commit message: Many refinements
Parts:
- added C9: 1000uF, Capacitor_SMD:CP_Elec_5x4.4, symbol Device:CP_Small
- added D7: WS2811, LED_THT:LED_D5.0mm-4_RGB, symbol LED:NeoPixel_THT
- added R7: 500R, Resistor_SMD:R_0805_2012Metric_Pad1.15x1.40mm_HandSolder, symbol Device:R_Small
- D1, D2, D3, D4, D5, D6: value NeoPixel -> WS2811
- J11, J12: value Conn_01x06 -> IDC_2x3
Connections:
- wire segments 95 -> 107
Other:
- note added: "This is a simple I2C port expander to reduce the number\nof connections back to the main board."
- note added: "Using a chain of NeoPixels as indicators, to reduce\nthe number of connections back to the main board."

Commit message: Various changes
Connections:
- wire segments 107 -> 106
Changed lines of the file:
@@
 NoConn ~ 5075 4950
 Wire Wire Line
-	4275 4250 4075 4250
-Wire Wire Line
-	4275 4350 4075 4350
-Wire Wire Line
-	4275 4450 4075 4450
+	4275 4250 3925 4250
+Wire Wire Line
+	4275 4350 3925 4350
+Wire Wire Line
+	4275 4450 3925 4450
 $Comp
 L Connector_Generic:Conn_01x06 J11
@@
 Text Label 1675 2625 0    39   ~ 0
 Panel_LED
-Text Label 4075 4250 2    39   ~ 0
+Text Label 3925 4250 0    39   ~ 0
 Button_SCL
-Text Label 4075 4350 2    39   ~ 0
+Text Label 3925 4350 0    39   ~ 0
 Button_SDA
-Text Label 4075 4450 2    39   ~ 0
+Text Label 3925 4450 0    39   ~ 0
 Button_INT
 Text Label 1675 2325 0    39   ~ 0
@@
 $EndComp
 Wire Wire Line
-	5225 2200 5200 2200
-Wire Wire Line
 	5200 2200 5200 2300
 Wire Wire Line
@@
 	1    0    0    -1
 $EndComp
-Text Label 5225 2200 0    39   ~ 0
+Text Label 5200 2200 0    39   ~ 0
 Panel_LED
 $EndSCHEMATC

Commit message: Various updates and tweaks
Parts:
- C9: value 1000uF -> 220uF; footprint Capacitor_SMD:CP_Elec_5x4.4 -> Capacitor_SMD:CP_Elec_8x6.2; manf# (none) -> UCD1C221MCL6GS
- R7: footprint Resistor_SMD:R_0805_2012Metric_Pad1.15x1.40mm_HandSolder -> Resistor_SMD:R_0603_1608Metric_Pad1.05x0.95mm_HandSolder; manf# (none) -> RC0603FR-07510RL
- U6: footprint Package_SO:SOIC-16W_7.5x12.8mm_P1.27mm -> Package_SO:SOIC-16W_7.5x10.3mm_P1.27mm; manf# (none) -> TCA9534DWR

Commit message: Before trying a single-board
Parts:
- SW1, SW2, SW3, SW4, SW5, SW6: footprint Button_Switch_THT:SW_PUSH_6mm_H13mm -> Button_Switch_THT:SW_CK_D6R_SPST_12mm_H14.3mm; symbol Switch:SW_Push -> Switch:SW_CK_D6R_SPST
Changed lines of the file:
@@
 NoConn ~ 9950 2550
 $Comp
-L Switch:SW_Push SW1
+L Switch:SW_CK_D6R_SPST SW1
 U 1 1 5BAD9A26
 P 6975 4875
-F 0 "SW1" H 7000 4975 50  0000 L CNN
+F 0 "SW1" H 6975 4975 50  0000 C CNN
 F 1 "SW_Push" H 7275 4875 50  0000 L CNN
-F 2 "Button_Switch_THT:SW_PUSH_6mm_H13mm" H 6975 5075 50  0001 C CNN
+F 2 "Button_Switch_THT:SW_CK_D6R_SPST_12mm_H14.3mm" H 6975 5075 50  0001 C CNN
 F 3 "" H 6975 5075 50  0001 C CNN
 	1    6975 4875
@@
 	6150 4125 6775 4125
 $Comp
-L Switch:SW_Push SW2
+L Switch:SW_CK_D6R_SPST SW2
 U 1 1 5BADAA87
 P 6975 5050
-F 0 "SW2" H 7000 5150 50  0000 L CNN
+F 0 "SW2" H 6975 5150 50  0000 C CNN
 F 1 "SW_Push" H 7275 5050 50  0000 L CNN
-F 2 "Button_Switch_THT:SW_PUSH_6mm_H13mm" H 6975 5250 50  0001 C CNN
+F 2 "Button_Switch_THT:SW_CK_D6R_SPST_12mm_H14.3mm" H 6975 5250 50  0001 C CNN
 F 3 "" H 6975 5250 50  0001 C CNN
 	1    6975 5050
@@
 $EndComp
 $Comp
-L Switch:SW_Push SW3
+L Switch:SW_CK_D6R_SPST SW3
 U 1 1 5BADAABB
 P 6975 4125
-F 0 "SW3" H 7000 4225 50  0000 L CNN
+F 0 "SW3" H 6975 4225 50  0000 C CNN
 F 1 "SW_Push" H 7275 4125 50  0000 L CNN
-F 2 "Button_Switch_THT:SW_PUSH_6mm_H13mm" H 6975 4325 50  0001 C CNN
+F 2 "Button_Switch_THT:SW_CK_D6R_SPST_12mm_H14.3mm" H 6975 4325 50  0001 C CNN
 F 3 "" H 6975 4325 50  0001 C CNN
 	1    6975 4125
@@
 $EndComp
 $Comp
-L Switch:SW_Push SW4
+L Switch:SW_CK_D6R_SPST SW4
 U 1 1 5BADAAEF
 P 6975 4325
-F 0 "SW4" H 7000 4425 50  0000 L CNN
+F 0 "SW4" H 6975 4425 50  0000 C CNN
 F 1 "SW_Push" H 7275 4325 50  0000 L CNN
-F 2 "Button_Switch_THT:SW_PUSH_6mm_H13mm" H 6975 4525 50  0001 C CNN
+F 2 "Button_Switch_THT:SW_CK_D6R_SPST_12mm_H14.3mm" H 6975 4525 50  0001 C CNN
 F 3 "" H 6975 4525 50  0001 C CNN
 	1    6975 4325
@@
 $EndComp
 $Comp
-L Switch:SW_Push SW5
+L Switch:SW_CK_D6R_SPST SW5
 U 1 1 5BADAB27
 P 6975 4525
-F 0 "SW5" H 7000 4625 50  0000 L CNN
+F 0 "SW5" H 6975 4625 50  0000 C CNN
 F 1 "SW_Push" H 7275 4525 50  0000 L CNN
-F 2 "Button_Switch_THT:SW_PUSH_6mm_H13mm" H 6975 4725 50  0001 C CNN
+F 2 "Button_Switch_THT:SW_CK_D6R_SPST_12mm_H14.3mm" H 6975 4725 50  0001 C CNN
 F 3 "" H 6975 4725 50  0001 C CNN
 	1    6975 4525
@@
 Button_INT
 $Comp
-L Switch:SW_Push SW6
+L Switch:SW_CK_D6R_SPST SW6
 U 1 1 5BB45FCD
 P 6975 4700
-F 0 "SW6" H 7000 4800 50  0000 L CNN
+F 0 "SW6" H 6975 4800 50  0000 C CNN
 F 1 "SW_Push" H 7275 4700 50  0000 L CNN
-F 2 "Button_Switch_THT:SW_PUSH_6mm_H13mm" H 6975 4900 50  0001 C CNN
+F 2 "Button_Switch_THT:SW_CK_D6R_SPST_12mm_H14.3mm" H 6975 4900 50  0001 C CNN
 F 3 "" H 6975 4900 50  0001 C CNN
 	1    6975 4700
